File: OldRemote.kicad_sch (KiCad schematic)
At the start: 21 parts, among them J1 Tristate Selector, J2 12V Battery, Q1 BF494, SW1 SW_Push, SW2 SW_Push, U1 MC145026

Commit message: Update schematic
Connections:
- net at AE2.2, C2.2, C3.2: now also C3.1, Q1.1 (C)
Changed lines of the file:
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@@
   (junction (at 55.88 121.92) (diameter 0) (color 0 0 0 0)
   )
+  (junction (at 181.61 54.61) (diameter 0) (color 0 0 0 0)
+  )
   (junction (at 172.72 97.79) (diameter 0) (color 0 0 0 0)
   )
@@
   (junction (at 193.04 54.61) (diameter 0) (color 0 0 0 0)
   )
+  (junction (at 168.91 54.61) (diameter 0) (color 0 0 0 0)
+  )
   (junction (at 71.12 107.95) (diameter 0) (color 0 0 0 0)
   )
@@
     (stroke (width 0) (type default))
   )
+  (wire (pts (xy 168.91 54.61) (xy 168.91 59.69))
+    (stroke (width 0) (type default))
+  )
   (wire (pts (xy 92.71 107.95) (xy 92.71 110.49))
     (stroke (width 0) (type default))
@@
     (stroke (width 0) (type default))
   )
+  (wire (pts (xy 181.61 54.61) (xy 193.04 54.61))
+    (stroke (width 0) (type default))
+  )
   (wire (pts (xy 139.7 156.21) (xy 182.88 156.21))
     (stroke (width 0) (type default))
@@
     (stroke (width 0) (type default))
   )
+  (wire (pts (xy 168.91 59.69) (xy 181.61 59.69))
+    (stroke (width 0) (type default))
+  )
   (wire (pts (xy 166.37 97.79) (xy 172.72 97.79))
     (stroke (width 0) (type default))
@@
     (stroke (width 0) (type default))
   )
+  (wire (pts (xy 168.91 54.61) (xy 172.72 54.61))
+    (stroke (width 0) (type default))
+  )
   (wire (pts (xy 55.88 115.57) (xy 55.88 116.84))
     (stroke (width 0) (type default))
@@
     (stroke (width 0) (type default))
   )
-  (wire (pts (xy 160.02 54.61) (xy 172.72 54.61))
+  (wire (pts (xy 160.02 54.61) (xy 168.91 54.61))
     (stroke (width 0) (type default))
   )
@@
     (stroke (width 0) (type default))
   )
-  (wire (pts (xy 177.8 54.61) (xy 193.04 54.61))
+  (wire (pts (xy 177.8 54.61) (xy 181.61 54.61))
     (stroke (width 0) (type default))
   )
@@
     (stroke (width 0) (type default))
   )
+  (wire (pts (xy 181.61 59.69) (xy 181.61 54.61))
+    (stroke (width 0) (type default))
+  )
